Commit message: update readme

File: remote_control/master1/src/arm_control/models/ultron_v1.1_aa.urdf (robot description, URDF)
Before this commit: robot ultron_v1.1_aa, 7 links, 6 joints
Links:
- link link6: mass 0.620000 -> 0.640000

File: remote_control/master2/src/arm_control/models/ultron_v1.1_aa.urdf (robot description, URDF)
Before this commit: robot ultron_v1.1_aa, 7 links, 6 joints
Links:
- link link6: mass 0.650000 -> 0.640000

Commit message: update code

File: remote_control/master1/src/arm_control/models/ultron_v1.1_aa.urdf (robot description, URDF)
Before this commit: robot ultron_v1.1_aa, 7 links, 6 joints
Links:
- link link6: mass 0.640000 -> 0.680000
